File: hardware/interceptor.sch (KiCad schematic (older format))
At the start: 32 parts, among them IC1 ATMEGA1284P-P, K1 USB, P1 TAPEPORT, P2 CIA1, P3 KEYBOARD, P4 USER A, P5 USER B, SW1 RESET, SW2 BOOTLOADER, U1 7400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

Commit message: Hardware: Fixed Crosspoint switch and usb connector, routed usb traces
Parts:
- removed K1: USB, symbol CONN_3
- added P6: USB, symbol CONN_9
Connections:
- no-connect marks 6 -> 12
Other:
- moved on the sheet: P1
Changed lines of the file:
@@
 Sheet 1 1
 Title "Programmable C64 Keyboard Interceptor and Controller"
-Date "1 aug 2015"
+Date "3 aug 2015"
 Rev "1"
 Comp "Henning Bekel"
@@
 L VCC #PWR03
 U 1 1 55A76720
-P 6350 7500
-F 0 "#PWR03" H 6350 7600 30  0001 C CNN
-F 1 "VCC" H 6350 7600 30  0000 C CNN
-F 2 "" H 6350 7500 60  0000 C CNN
-F 3 "" H 6350 7500 60  0000 C CNN
-	1    6350 7500
+P 10350 6800
+F 0 "#PWR03" H 10350 6900 30  0001 C CNN
+F 1 "VCC" H 10350 6900 30  0000 C CNN
+F 2 "" H 10350 6800 60  0000 C CNN
+F 3 "" H 10350 6800 60  0000 C CNN
+	1    10350 6800
 	-1   0    0    1
 $EndComp
@@
 L PWR_FLAG #FLG04
 U 1 1 55A7672F
-P 6350 7400
-F 0 "#FLG04" H 6350 7495 30  0001 C CNN
-F 1 "PWR_FLAG" H 6350 7580 30  0000 C CNN
-F 2 "" H 6350 7400 60  0000 C CNN
-F 3 "" H 6350 7400 60  0000 C CNN
-	1    6350 7400
-	1    0    0    -1
-$EndComp
-Wire Wire Line
-	6350 7400 6350 7500
+P 10350 6700
+F 0 "#FLG04" H 10350 6795 30  0001 C CNN
+F 1 "PWR_FLAG" H 10350 6880 30  0000 C CNN
+F 2 "" H 10350 6700 60  0000 C CNN
+F 3 "" H 10350 6700 60  0000 C CNN
+	1    10350 6700
+	1    0    0    -1
+$EndComp
+Wire Wire Line
+	10350 6700 10350 6800
 $Comp
 L PWR_FLAG #FLG05
 U 1 1 55A767C3
-P 6650 7400
-F 0 "#FLG05" H 6650 7495 30  0001 C CNN
-F 1 "PWR_FLAG" H 6650 7580 30  0000 C CNN
-F 2 "" H 6650 7400 60  0000 C CNN
-F 3 "" H 6650 7400 60  0000 C CNN
-	1    6650 7400
+P 10650 6700
+F 0 "#FLG05" H 10650 6795 30  0001 C CNN
+F 1 "PWR_FLAG" H 10650 6880 30  0000 C CNN
+F 2 "" H 10650 6700 60  0000 C CNN
+F 3 "" H 10650 6700 60  0000 C CNN
+	1    10650 6700
 	1    0    0    -1
 $EndComp
@@
 L GND #PWR06
 U 1 1 55A767D2
-P 6650 7550
-F 0 "#PWR06" H 6650 7550 30  0001 C CNN
-F 1 "GND" H 6650 7480 30  0001 C CNN
-F 2 "" H 6650 7550 60  0000 C CNN
-F 3 "" H 6650 7550 60  0000 C CNN
-	1    6650 7550
-	1    0    0    -1
-$EndComp
-Wire Wire Line
-	6650 7400 6650 7550
+P 10650 6850
+F 0 "#PWR06" H 10650 6850 30  0001 C CNN
+F 1 "GND" H 10650 6780 30  0001 C CNN
+F 2 "" H 10650 6850 60  0000 C CNN
+F 3 "" H 10650 6850 60  0000 C CNN
+	1    10650 6850
+	1    0    0    -1
+$EndComp
+Wire Wire Line
+	10650 6700 10650 6850
 $Comp
 L GND #PWR07
@@
 L CONN_2 P1
 U 1 1 55A772B0
-P 1300 1150
-F 0 "P1" V 1250 1150 40  0000 C CNN
-F 1 "TAPEPORT" V 1350 1150 40  0000 C CNN
-F 2 "" H 1300 1150 60  0000 C CNN
-F 3 "" H 1300 1150 60  0000 C CNN
-	1    1300 1150
-	1    0    0    -1
-$EndComp
-Text Label 950  1050 2    60   ~ 0
+P 1250 1000
+F 0 "P1" V 1200 1000 40  0000 C CNN
+F 1 "TAPEPORT" V 1300 1000 40  0000 C CNN
+F 2 "" H 1250 1000 60  0000 C CNN
+F 3 "" H 1250 1000 60  0000 C CNN
+	1    1250 1000
+	1    0    0    -1
+$EndComp
+Text Label 900  900  2    60   ~ 0
 CS
-Text Label 950  1250 2    60   ~ 0
+Text Label 900  1100 2    60   ~ 0
 CD
 $Comp
@@
 Text Label 2300 3900 2    60   ~ 0
 ~RESET
-$Comp
-L CONN_3 K1
-U 1 1 55B37C90
-P 1300 700
-F 0 "K1" V 1250 700 50  0000 C CNN
-F 1 "USB" V 1350 700 40  0000 C CNN
-F 2 "" H 1300 700 60  0000 C CNN
-F 3 "" H 1300 700 60  0000 C CNN
-	1    1300 700
-	1    0    0    -1
-$EndComp
-Text Label 950  700  2    60   ~ 0
-D+
-Text Label 950  600  2    60   ~ 0
-D-
-$Comp
-L GND #PWR043
-U 1 1 55B37CAF
-P 950 800
-F 0 "#PWR043" H 950 800 30  0001 C CNN
-F 1 "GND" H 950 730 30  0001 C CNN
-F 2 "" H 950 800 60  0000 C CNN
-F 3 "" H 950 800 60  0000 C CNN
-	1    950  800
-	0    1    1    0
-$EndComp
 Text Label 5700 6700 0    60   ~ 0
 D-
@@
 $EndComp
 $Comp
-L VCC #PWR044
+L VCC #PWR043
 U 1 1 55B38389
 P 10750 4750
-F 0 "#PWR044" H 10750 4850 30  0001 C CNN
+F 0 "#PWR043" H 10750 4850 30  0001 C CNN
 F 1 "VCC" H 10750 4850 30  0000 C CNN
 F 2 "" H 10750 4750 60  0000 C CNN
@@
 $EndComp
 $Comp
-L GND #PWR045
+L GND #PWR044
 U 1 1 55B3838F
 P 10750 5150
-F 0 "#PWR045" H 10750 5150 30  0001 C CNN
+F 0 "#PWR044" H 10750 5150 30  0001 C CNN
 F 1 "GND" H 10750 5080 30  0001 C CNN
 F 2 "" H 10750 5150 60  0000 C CNN
@@
 $EndComp
 $Comp
-L VCC #PWR046
+L VCC #PWR045
 U 1 1 55B387FF
 P 5200 6200
-F 0 "#PWR046" H 5200 6300 30  0001 C CNN
+F 0 "#PWR045" H 5200 6300 30  0001 C CNN
 F 1 "VCC" H 5200 6300 30  0000 C CNN
 F 2 "" H 5200 6200 60  0000 C CNN
@@
 $EndComp
 $Comp
-L GND #PWR047
+L GND #PWR046
 U 1 1 55B38813
 P 5200 7200
-F 0 "#PWR047" H 5200 7200 30  0001 C CNN
+F 0 "#PWR046" H 5200 7200 30  0001 C CNN
 F 1 "GND" H 5200 7130 30  0001 C CNN
 F 2 "" H 5200 7200 60  0000 C CNN
@@
 $EndComp
 $Comp
-L GND #PWR048
+L GND #PWR047
 U 1 1 55B38825
 P 4900 7100
-F 0 "#PWR048" H 4900 7100 30  0001 C CNN
+F 0 "#PWR047" H 4900 7100 30  0001 C CNN
 F 1 "GND" H 4900 7030 30  0001 C CNN
 F 2 "" H 4900 7100 60  0000 C CNN
@@
 NoConn ~ 11100 6100
 $Comp
-L GND #PWR049
+L GND #PWR048
 U 1 1 55B4B074
 P 9900 6000
-F 0 "#PWR049" H 9900 6000 30  0001 C CNN
+F 0 "#PWR048" H 9900 6000 30  0001 C CNN
 F 1 "GND" H 9900 5930 30  0001 C CNN
 F 2 "" H 9900 6000 60  0000 C CNN
@@
 $EndComp
 $Comp
-L GND #PWR050
+L GND #PWR049
 U 1 1 55B4B08B
 P 9900 6200
-F 0 "#PWR050" H 9900 6200 30  0001 C CNN
+F 0 "#PWR049" H 9900 6200 30  0001 C CNN
 F 1 "GND" H 9900 6130 30  0001 C CNN
 F 2 "" H 9900 6200 60  0000 C CNN
@@
 MR
 $Comp
-L GND #PWR051
+L GND #PWR050
 U 1 1 55B68DDD
 P 2650 2600
-F 0 "#PWR051" H 2650 2600 30  0001 C CNN
+F 0 "#PWR050" H 2650 2600 30  0001 C CNN
 F 1 "GND" H 2650 2530 30  0001 C CNN
 F 2 "" H 2650 2600 60  0000 C CNN
@@
 $EndComp
 $Comp
-L GND #PWR?
+L GND #PWR051
 U 1 1 55BD089A
 P 3350 2650
-F 0 "#PWR?" H 3350 2650 30  0001 C CNN
+F 0 "#PWR051" H 3350 2650 30  0001 C CNN
 F 1 "GND" H 3350 2580 30  0001 C CNN
 F 2 "" H 3350 2650 60  0000 C CNN
@@
 	1    0    0    -1
 $EndComp
+$Comp
+L CONN_9 P6
+U 1 1 55BF1030
+P 6350 7000
+F 0 "P6" V 6300 7000 60  0000 C CNN
+F 1 "USB" V 6400 7000 60  0000 C CNN
+F 2 "" H 6350 7000 60  0000 C CNN
+F 3 "" H 6350 7000 60  0000 C CNN
+	1    6350 7000
+	-1   0    0    1
+$EndComp
+NoConn ~ 6700 7400
+NoConn ~ 6700 7100
+Text Label 6700 7300 0    60   ~ 0
+D-
+Text Label 6700 7200 0    60   ~ 0
+D+
+$Comp
+L GND #PWR052
+U 1 1 55BF10BD
+P 6700 7000
+F 0 "#PWR052" H 6700 7000 30  0001 C CNN
+F 1 "GND" H 6700 6930 30  0001 C CNN
+F 2 "" H 6700 7000 60  0000 C CNN
+F 3 "" H 6700 7000 60  0000 C CNN
+	1    6700 7000
+	0    -1   -1   0
+$EndComp
+NoConn ~ 6700 6900
+NoConn ~ 6700 6800
+NoConn ~ 6700 6700
+NoConn ~ 6700 6600
 $EndSCHEMATC

Commit message: Hardware: First serious draft of pcb layout
Parts:
- removed C13, C7, C8, C9: 100nF, ~, symbol C
- removed P4: USER A, symbol CONN_8
- removed P5: USER B, symbol CONN_8
- added JP1: JUMPER, ~, symbol JUMPER
- added P4: USER, symbol CONN_8X2
Connections:
- net UA0: now also P4.1
- net UA1: now also P4.3
- net UA2: now also P4.5
- net UA3: now also P4.7
- net UA4: now also P4.9
- net UA5: now also P4.11
- net UA6: now also P4.13
- net UA7: now also P4.15
- net UB0: now also P4.2
- net UB1: now also P4.4
- net UB2: now also P4.6
- net UB3: now also P4.8
- net UB4: now also P4.10
- net UB5: now also P4.12
- net UB6: now also P4.14
- net UB7: now also P4.16
- net VCC: now also JP1.2; no longer P2.4 (P4), P3.4 (P4)
- new net EXTVCC: JP1.1, P2.4 (P4)
- no-connect marks 12 -> 13
Other:
- note added: "8x8 Crosspoint Switch"
- note added: "Connectors"
- note added: "Counters for serial Matrix scan\n"
- note added: "Matrix scan multiplexers"
- note added: "Microprocessor"
- note added: "Negative power supply"
- note added: "Power flags"
- note added: "Reset Signal for Counters"
- note added: "Reset/Bootloader Buttons"
- note added: "Stabilizing caps"
- note added: "Unused gates"
- moved on the sheet: C10, C11, C12, C4, C5, P1, P2, P3, P6, SW1, SW2, U1A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
